File: pcb/joey.brd (EAGLE design)
At the start: 42.8 x 49.8 mm, 62 parts, among them J1 AVR_SPI_PRG_6PTH, U1 ATMEGA168, U2 TMP102, X1 USB-MICROB, Y1 13.56M

Commit message: Fixed the varactor grounding bug in v1.0
Connections:
- removed net SMV1247-1: SMV1232-1.AN, SMV1236-1.2
- net GND: now also SMV1232-1.AN, SMV1236-1.2
Routing:
- net VCC: track 150.0 -> 152.5 mm
- net SMV1247-1: track 1.92 -> 0.00 mm
- net GND: vias 84 -> 86
Changed lines of the file:
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@@
 <via x="25.654" y="44.196" extent="1-16" drill="0.508"/>
 <via x="24.384" y="45.466" extent="1-16" drill="0.508"/>
+<contactref element="SMV1232-1" pad="AN"/>
+<contactref element="SMV1236-1" pad="2"/>
+<via x="5.588" y="24.892" extent="1-16" drill="0.508"/>
+<via x="7.366" y="24.892" extent="1-16" drill="0.508"/>
 </signal>
 <signal name="VCC">
@@
 <wire x1="5.588" y1="12.534" x2="4.738" y2="12.534" width="0.3048" layer="1"/>
 <wire x1="4.738" y1="12.534" x2="4.318" y2="12.954" width="0.3048" layer="1"/>
-<wire x1="4.318" y1="12.954" x2="4.318" y2="24.13" width="0.3048" layer="1"/>
-<wire x1="4.318" y1="24.13" x2="4.826" y2="24.638" width="0.3048" layer="1"/>
-<wire x1="4.826" y1="24.638" x2="8.04" y2="24.638" width="0.3048" layer="1"/>
-<wire x1="8.04" y1="24.638" x2="9.056" y2="23.622" width="0.3048" layer="1"/>
+<wire x1="4.318" y1="12.954" x2="4.318" y2="25.146" width="0.3048" layer="1"/>
+<wire x1="4.318" y1="25.146" x2="5.08" y2="25.908" width="0.3048" layer="1"/>
+<wire x1="5.08" y1="25.908" x2="8.128" y2="25.908" width="0.3048" layer="1"/>
 <wire x1="9.056" y1="23.622" x2="9.144" y2="23.622" width="0.3048" layer="1"/>
 <wire x1="7.906" y1="12.176" x2="11.906" y2="12.176" width="0.3048" layer="1"/>
@@
 <wire x1="32.462" y1="27.14" x2="32.462" y2="27.559" width="0.4064" layer="1"/>
 <wire x1="32.462" y1="27.559" x2="32.462" y2="29.96" width="0.4064" layer="1"/>
+<wire x1="8.128" y1="25.908" x2="8.89" y2="25.146" width="0.3048" layer="1"/>
+<wire x1="8.89" y1="25.146" x2="8.89" y2="23.876" width="0.3048" layer="1"/>
+<wire x1="8.89" y1="23.876" x2="9.144" y2="23.622" width="0.3048" layer="1"/>
 </signal>
 <signal name="N$1">
@@
 <wire x1="30.926" y1="19.558" x2="32.932" y2="19.558" width="0.4064" layer="1"/>
 </signal>
-<signal name="SMV1247-1">
-<contactref element="SMV1232-1" pad="AN"/>
-<contactref element="SMV1236-1" pad="2"/>
-<wire x1="5.588" y1="23.756" x2="7.016" y2="23.756" width="0.3048" layer="1"/>
-<wire x1="7.016" y1="23.756" x2="7.366" y2="23.406" width="0.3048" layer="1"/>
-</signal>
 <signal name="COARSE">
