File: pcb/joey.brd (EAGLE design)
At the start: 42.8 x 49.8 mm, 62 parts, among them J1 AVR_SPI_PRG_6PTH, U1 ATMEGA168, U2 TMP102, X1 USB-MICROB, Y1 13.56M

Commit message: Finished rev2 of Joey, submission to CCC at this SHA1
Parts:
- removed U2: TMP102, SparkFun:SOT563
- added U$11: (no value), jonsowman:CUSF_LOGO_LARGE
- added U$12: TMP100, jonsowman:SOT23-6
- moved LEDA 0.25 mm to (12.2, 29.0)
- moved LEDB 0.25 mm to (12.2, 27.2)
Connections:
- net GND: now also U$12.2, U$12.5; no longer U2.2, U2.4
- net I2C_SCL: now also U$12.1; no longer U2.1
- net I2C_SDA: now also U$12.6; no longer U2.6
- net VCC: now also U$12.4; no longer U2.5
Routing:
- net GND: track 122.5 -> 103.0 mm, vias 86 -> 85
- net I2C_SDA: track 8.34 -> 15.6 mm
- net I2C_SCL: track 12.7 -> 9.21 mm, vias 2 -> 0
- net VCC: track 152.5 -> 150.3 mm
Other:
- board text added: "OCT '12"
- board text added: "cusf.co.uk"
- board text removed: "CU SPACEFLIGHT"
- board text removed: "MAR '12"
- board text removed: "http://cusf.co.uk"
